File: Project_Metronome/MetronomeSMD.sch (EAGLE design)
At the start: 45 parts

Commit message: better eagle files
Parts:
- added .: (no value), adafruit:PINHD-1X3CB
- JP1: device adafruit:PINHD-1X3CB -> adafruit:PINHD-1X6LOCK
- renumbered JP17 to ..., JP18 to ....., JP2 to .., LED1 to RED, LED2 to GREEN, LED3 to LED, R1 to 1, R10 to 17, R11 to 16, R12 to 15, R13 to 13, R14 to 12, R15 to 11, R16 to 10, R2 to 2, R3 to 3, R4 to 4, R5 to 6, R6 to 7, R7 to 8, R8 to 9, R9 to 18
Connections:
- net GND: now also JP1.3
- net N$22: now also JP1.4
- net N$24: now also JP1.5
- net N$27: now also JP1.6
- net N$5: now also JP1.1
- net VDD: now also ..1, ..2, ..3; no longer JP1.1, JP1.3
