File: Project_Metronome/Schematics/ece411-t14-MetroKnome.sch (EAGLE design)
At the start: 52 parts, among them Q2 BC846

Commit message: Add files via upload
Other:
- note added: "remove pull-up resistors from encoder and populate main PCB"
- note removed: "pull-up resistors are located off board with the encoder"
- moved on the sheet: 12, 13, G1, G2, LED, Q1, Q2, R22, SJ1, SJ3
